File: cad/goldfish.sch (KiCad schematic (older format))
At the start: 22 parts, among them J1 USB-C, J2 01x02, J3 01x12, J4 01x12, J5 01x05, U1 ATmega32U4, X1 16MHz

Commit message: Rev. A - Changed footprint of C6 from 0402 to 0603 to reduce component cost
Parts:
- C6: footprint Capacitors_SMD:C_0402 -> Capacitors_SMD:C_0603
Changed lines of the file:
@@
 LIBS:valves
 LIBS:atmega32u4-ep
-LIBS:goldfish-cache
 EELAYER 25 0
 EELAYER END
@@
 Sheet 1 1
 Title "Goldfish"
-Date "2017-12-12"
-Rev "0"
+Date "2017-12-20"
+Rev "A"
 Comp ""
 Comment1 ""
@@
 F 0 "C6" H 6625 1250 50  0000 L CNN
 F 1 "4u7" H 6625 1050 50  0000 L CNN
-F 2 "Capacitors_SMD:C_0402" H 6638 1000 50  0001 C CNN
+F 2 "Capacitors_SMD:C_0603" H 6638 1000 50  0001 C CNN
 F 3 "" H 6600 1150 50  0001 C CNN
 	1    6600 1150

Commit message: Rev. B - Fixed split keyboard issue and tidied up layout
Parts:
- added D1: D_Schottky, Diodes_SMD:D_PowerDI-123, symbol D_Schottky
Connections:
- net labels added: VBUS
- wire segments 157 -> 163
Changed lines of the file:
@@
 Title "Goldfish"
 Date "2017-12-20"
-Rev "A"
+Rev "B"
 Comp ""
 Comment1 ""
@@
 $EndComp
 $Comp
-L VCC #PWR05
-U 1 1 5A285F3B
-P 3000 1200
-F 0 "#PWR05" H 3000 1050 50  0001 C CNN
-F 1 "VCC" H 3000 1350 50  0000 C CNN
-F 2 "" H 3000 1200 50  0001 C CNN
-F 3 "" H 3000 1200 50  0001 C CNN
-	1    3000 1200
-	1    0    0    -1
-$EndComp
-$Comp
 L ATMEGA32U4-EP U1
 U 1 1 5A28636A
@@
 $EndComp
 $Comp
-L GND #PWR06
+L GND #PWR05
 U 1 1 5A28642D
 P 8400 5150
-F 0 "#PWR06" H 8400 4900 50  0001 C CNN
+F 0 "#PWR05" H 8400 4900 50  0001 C CNN
 F 1 "GND" H 8400 5000 50  0000 C CNN
 F 2 "" H 8400 5150 50  0001 C CNN
@@
 $EndComp
 $Comp
-L GND #PWR07
+L GND #PWR06
 U 1 1 5A287391
 P 6700 3000
-F 0 "#PWR07" H 6700 2750 50  0001 C CNN
+F 0 "#PWR06" H 6700 2750 50  0001 C CNN
 F 1 "GND" H 6700 2850 50  0000 C CNN
 F 2 "" H 6700 3000 50  0001 C CNN
@@
 $EndComp
 $Comp
-L VCC #PWR08
+L VCC #PWR07
 U 1 1 5A288631
 P 7400 1500
-F 0 "#PWR08" H 7400 1350 50  0001 C CNN
+F 0 "#PWR07" H 7400 1350 50  0001 C CNN
 F 1 "VCC" H 7400 1650 50  0000 C CNN
 F 2 "" H 7400 1500 50  0001 C CNN
@@
 $EndComp
 $Comp
-L GND #PWR09
+L GND #PWR08
 U 1 1 5A288F15
 P 7900 3900
-F 0 "#PWR09" H 7900 3650 50  0001 C CNN
+F 0 "#PWR08" H 7900 3650 50  0001 C CNN
 F 1 "GND" H 7900 3750 50  0000 C CNN
 F 2 "" H 7900 3900 50  0001 C CNN
@@
 D-
 $Comp
-L VCC #PWR010
+L VCC #PWR09
 U 1 1 5A28A25C
-P 8600 1350
-F 0 "#PWR010" H 8600 1200 50  0001 C CNN
-F 1 "VCC" H 8600 1500 50  0000 C CNN
-F 2 "" H 8600 1350 50  0001 C CNN
-F 3 "" H 8600 1350 50  0001 C CNN
-	1    8600 1350
+P 9500 1350
+F 0 "#PWR09" H 9500 1200 50  0001 C CNN
+F 1 "VCC" H 9500 1500 50  0000 C CNN
+F 2 "" H 9500 1350 50  0001 C CNN
+F 3 "" H 9500 1350 50  0001 C CNN
+	1    9500 1350
 	1    0    0    -1
 $EndComp
@@
 $EndComp
 $Comp
-L GND #PWR011
+L GND #PWR010
 U 1 1 5A28A75C
 P 7900 4700
-F 0 "#PWR011" H 7900 4450 50  0001 C CNN
+F 0 "#PWR010" H 7900 4450 50  0001 C CNN
 F 1 "GND" H 7900 4550 50  0000 C CNN
 F 2 "" H 7900 4700 50  0001 C CNN
@@
 PE6
 $Comp
-L GND #PWR012
+L GND #PWR011
 U 1 1 5A28C2FC
 P 10750 4000
-F 0 "#PWR012" H 10750 3750 50  0001 C CNN
+F 0 "#PWR011" H 10750 3750 50  0001 C CNN
 F 1 "GND" H 10750 3850 50  0000 C CNN
 F 2 "" H 10750 4000 50  0001 C CNN
@@
 PD2
 $Comp
-L GND #PWR013
+L GND #PWR012
 U 1 1 5A28F1F6
 P 4550 3650
-F 0 "#PWR013" H 4550 3400 50  0001 C CNN
+F 0 "#PWR012" H 4550 3400 50  0001 C CNN
 F 1 "GND" H 4550 3500 50  0000 C CNN
 F 2 "" H 4550 3650 50  0001 C CNN
@@
 PF7
 $Comp
-L VCC #PWR014
+L VCC #PWR013
 U 1 1 5A293402
-P 4950 3150
-F 0 "#PWR014" H 4950 3000 50  0001 C CNN
-F 1 "VCC" H 4950 3300 50  0000 C CNN
-F 2 "" H 4950 3150 50  0001 C CNN
-F 3 "" H 4950 3150 50  0001 C CNN
-	1    4950 3150
-	1    0    0    -1
+P 5050 3550
+F 0 "#PWR013" H 5050 3400 50  0001 C CNN
+F 1 "VCC" H 5050 3700 50  0000 C CNN
+F 2 "" H 5050 3550 50  0001 C CNN
+F 3 "" H 5050 3550 50  0001 C CNN
+	1    5050 3550
+	0    -1   -1   0
 $EndComp
 Text Label 7100 1800 2    60   ~ 0
@@
 NoConn ~ 10350 3500
 $Comp
-L VCC #PWR015
+L VCC #PWR014
 U 1 1 5A296654
 P 5000 800
-F 0 "#PWR015" H 5000 650 50  0001 C CNN
+F 0 "#PWR014" H 5000 650 50  0001 C CNN
 F 1 "VCC" H 5000 950 50  0000 C CNN
 F 2 "" H 5000 800 50  0001 C CNN
@@
 $EndComp
 $Comp
-L GND #PWR016
+L GND #PWR015
 U 1 1 5A296BBF
 P 5000 1500
-F 0 "#PWR016" H 5000 1250 50  0001 C CNN
+F 0 "#PWR015" H 5000 1250 50  0001 C CNN
 F 1 "GND" H 5000 1350 50  0000 C CNN
 F 2 "" H 5000 1500 50  0001 C CNN
 F 3 "" H 5000 1500 50  0001 C CNN
 	1    5000 1500
-	1    0    0    -1
-$EndComp
-$Comp
-L VCC #PWR017
-U 1 1 5A29A6F8
-P 7900 2900
-F 0 "#PWR017" H 7900 2750 50  0001 C CNN
-F 1 "VCC" H 7900 3050 50  0000 C CNN
-F 2 "" H 7900 2900 50  0001 C CNN
-F 3 "" H 7900 2900 50  0001 C CNN
-	1    7900 2900
 	1    0    0    -1
 $EndComp
@@
 	8500 4950 8500 5050
 Wire Wire Line
-	6300 1300 6300 1400
-Wire Wire Line
-	6300 1000 6300 900
-Connection ~ 6300 900
-Connection ~ 6300 1400
-Wire Wire Line
 	2800 2500 3300 2500
 Wire Wire Line
@@
 Wire Wire Line
 	9300 1450 9300 1550
-Connection ~ 8950 1450
 Wire Wire Line
 	9050 1450 9050 1550
-Connection ~ 8700 1450
-Wire Wire Line
-	8950 1450 8950 1550
-Wire Wire Line
-	8700 1450 8700 1550
-Wire Wire Line
-	8600 1450 9400 1450
-Wire Wire Line
-	8600 1350 8600 1450
+Wire Wire Line
+	8950 1450 9500 1450
 Wire Wire Line
 	1800 4200 1800 4300
@@
 	2800 1200 2800 1600
 Wire Wire Line
-	2700 1300 3000 1300
+	2700 1300 3100 1300
 Connection ~ 2800 1300
 Wire Wire Line
@@
 	4950 4650 4950 4750
 Wire Wire Line
-	4950 3250 5350 3250
-Wire Wire Line
 	4550 3350 5350 3350
 Wire Wire Line
 	5250 3450 5350 3450
 Wire Wire Line
-	4950 3550 5350 3550
+	5050 3550 5350 3550
 Wire Wire Line
 	5250 3650 5350 3650
@@
 	4550 3350 4550 3650
 Connection ~ 4550 3550
-Wire Wire Line
-	4950 3150 4950 3550
-Connection ~ 4950 3250
 Connection ~ 4550 3450
 Wire Wire Line
@@
 Connection ~ 5700 1400
 Wire Wire Line
-	6000 1400 6000 1300
-Connection ~ 6000 1400
-Wire Wire Line
 	6600 900  6600 1000
 Wire Wire Line
-	5000 900  6600 900
-Wire Wire Line
-	6000 900  6000 1000
+	5000 900  6000 900
 Wire Wire Line
 	5700 900  5700 1000
-Connection ~ 6000 900
 Wire Wire Line
 	5400 900  5400 1000
@@
 Text Notes 700  7600 0    60   ~ 0
 Released under the Creative Commons Attribution Share-Alike 4.0 License\nhttps://creativecommons.org/licenses/by-sa/4.0/\n\nOriginal Arduino Mini Design by Team Arduino\nArduino Pro Mini Design by Spark Fun Electronics\nPro Micro Design by Spark Fun Electronics\nGoldfish Design by Dr Derivative
+$Comp
+L VBUS #PWR016
+U 1 1 5A78C3BD
+P 3000 1200
+F 0 "#PWR016" H 3000 1050 50  0001 C CNN
+F 1 "VBUS" H 3000 1350 50  0000 C CNN
+F 2 "" H 3000 1200 50  0001 C CNN
+F 3 "" H 3000 1200 50  0001 C CNN
+	1    3000 1200
+	1    0    0    -1
+$EndComp
+$Comp
+L VBUS #PWR017
+U 1 1 5A78C8B6
+P 7900 2900
+F 0 "#PWR017" H 7900 2750 50  0001 C CNN
+F 1 "VBUS" H 7900 3050 50  0000 C CNN
+F 2 "" H 7900 2900 50  0001 C CNN
+F 3 "" H 7900 2900 50  0001 C CNN
+	1    7900 2900
+	1    0    0    -1
+$EndComp
+$Comp
+L VBUS #PWR018
+U 1 1 5A78D027
+P 8600 1350
+F 0 "#PWR018" H 8600 1200 50  0001 C CNN
+F 1 "VBUS" H 8600 1500 50  0000 C CNN
+F 2 "" H 8600 1350 50  0001 C CNN
+F 3 "" H 8600 1350 50  0001 C CNN
+	1    8600 1350
+	1    0    0    -1
+$EndComp
+Wire Wire Line
+	8700 1550 8700 1450
+Wire Wire Line
+	8700 1450 8600 1450
+Wire Wire Line
+	8600 1450 8600 1350
+Wire Wire Line
+	9500 1450 9500 1350
+Connection ~ 9400 1450
+Wire Wire Line
+	8950 1450 8950 1550
+$Comp
+L D_Schottky D1
+U 1 1 5A78E24C
+P 3250 1300
+F 0 "D1" H 3250 1400 50  0000 C CNN
+F 1 "D_Schottky" H 3250 1200 50  0000 C CNN
+F 2 "Diodes_SMD:D_PowerDI-123" H 3250 1300 50  0001 C CNN
+F 3 "" H 3250 1300 50  0001 C CNN
+	1    3250 1300
+	-1   0    0    1
+$EndComp
+Connection ~ 3000 1300
+Wire Wire Line
+	3400 1300 3700 1300
+Wire Wire Line
+	3700 1300 3700 1200
+$Comp
+L VCC #PWR019
+U 1 1 5A78E470
+P 3700 1200
+F 0 "#PWR019" H 3700 1050 50  0001 C CNN
+F 1 "VCC" H 3700 1350 50  0000 C CNN
+F 2 "" H 3700 1200 50  0001 C CNN
+F 3 "" H 3700 1200 50  0001 C CNN
+	1    3700 1200
+	1    0    0    -1
+$EndComp
+$Comp
+L PWR_FLAG #FLG020
+U 1 1 5A79EAD6
+P 3500 1200
+F 0 "#FLG020" H 3500 1275 50  0001 C CNN
+F 1 "PWR_FLAG" H 3350 1350 50  0000 C CNN
+F 2 "" H 3500 1200 50  0001 C CNN
+F 3 "" H 3500 1200 50  0001 C CNN
+	1    3500 1200
+	1    0    0    -1
+$EndComp
+Wire Wire Line
+	3500 1200 3500 1300
+Connection ~ 3500 1300
+$Comp
+L VBUS #PWR021
+U 1 1 5A7A408A
+P 5050 3250
+F 0 "#PWR021" H 5050 3100 50  0001 C CNN
+F 1 "VBUS" H 5050 3400 50  0000 C CNN
+F 2 "" H 5050 3250 50  0001 C CNN
+F 3 "" H 5050 3250 50  0001 C CNN
+	1    5050 3250
+	0    -1   -1   0
+$EndComp
+Wire Wire Line
+	5050 3250 5350 3250
+Wire Wire Line
+	6000 900  6000 1000
+Wire Wire Line
+	6000 1400 6000 1300
+Wire Wire Line
+	6300 1400 6300 1300
+Wire Wire Line
+	6300 1000 6300 900
+Wire Wire Line
+	6200 900  6600 900
+Wire Wire Line
+	6200 900  6200 800
+Connection ~ 6300 900
+Connection ~ 6000 1400
+Connection ~ 6300 1400
+$Comp
+L VBUS #PWR?
+U 1 1 5A7A4C4A
+P 6200 800
+F 0 "#PWR?" H 6200 650 50  0001 C CNN
+F 1 "VBUS" H 6200 950 50  0000 C CNN
+F 2 "" H 6200 800 50  0001 C CNN
+F 3 "" H 6200 800 50  0001 C CNN
+	1    6200 800
+	1    0    0    -1
+$EndComp
 $EndSCHEMATC

Commit message: Rev. C - Changed bottom pins for Elite-C compatibility
Parts:
- added R6: 10k, Resistor_SMD:R_0402_1005Metric, symbol Device:R
- C1, C10, C2, C3, C4, C5, C7, C8, C9: footprint Capacitors_SMD:C_0402 -> Capacitor_SMD:C_0402_1005Metric; symbol C -> Device:C
- C6: footprint Capacitors_SMD:C_0603 -> Capacitor_SMD:C_0402_1005Metric; symbol C -> Device:C
- D1: footprint Diodes_SMD:D_PowerDI-123 -> Diode_SMD:D_PowerDI-123; symbol D_Schottky -> Device:D_Schottky
- J1: footprint USB Type-C:CX70M-24P1 -> usb-type-c:CX70M-24P1; symbol USB_C_Receptacle -> goldfish-rescue:USB_C_Receptacle-Connector
- J2: footprint Pins:Pins2 -> pins:Pins2; symbol Conn_01x02 -> Connector_Generic:Conn_01x02
- J3, J4: footprint Pins:Pins12 -> pins:Pins12; symbol Conn_01x12 -> Connector_Generic:Conn_01x12
- J5: footprint Pins:Pins5 -> pins:Pins5; symbol Conn_01x05 -> Connector_Generic:Conn_01x05
- R1, R2, R3, R4, R5: footprint Resistors_SMD:R_0402 -> Resistor_SMD:R_0402_1005Metric; symbol R -> Device:R
- U1: footprint Housings_DFN_QFN:QFN-44-1EP_7x7mm_Pitch0.5mm -> Package_DFN_QFN:QFN-44-1EP_7x7mm_P0.5mm_EP5.2x5.2mm; symbol ATMEGA32U4-EP -> atmega32u4-ep:ATMEGA32U4-EP
- X1: footprint Crystals:Crystal_SMD_SeikoEpson_FA238-4pin_3.2x2.5mm -> Crystal:Crystal_SMD_SeikoEpson_FA238-4Pin_3.2x2.5mm; symbol Crystal_GND24 -> Device:Crystal_GND24
Connections:
- net labels added: PD5
- net labels removed: PD6
- wire segments 163 -> 206
Other:
- note added: "Released under the Creative Commons Attribution Share-Alike 4.0 License\nhttps://creativecommons.org/licenses/by-sa/4.0/\n\nOriginal Arduino Mini Design by Team Arduino\nArduino Pro Mini Design by Spark Fun Electronics\nPro Micro Design by Spark Fun Electronics\nGoldfish Design by dr_derivative"
- note removed: "Released under the Creative Commons Attribution Share-Alike 4.0 License\nhttps://creativecommons.org/licenses/by-sa/4.0/\n\nOriginal Arduino Mini Design by Team Arduino\nArduino Pro Mini Design by Spark Fun Electronics\nPro Micro Design by Spark Fun Electronics\nGoldfish Design by Dr Derivative"

Commit message: Fixed missing goldfish-rescue file error
Parts:
- J1: symbol goldfish-rescue:USB_C_Receptacle-Connector -> Connector:USB_C_Receptacle
Connections:
- wire segments 206 -> 195
Changed lines of the file:
@@
 L power:GND #PWR01
 U 1 1 5A284D23
-P 2500 4400
-F 0 "#PWR01" H 2500 4150 50  0001 C CNN
-F 1 "GND" H 2500 4250 50  0000 C CNN
-F 2 "" H 2500 4400 50  0001 C CNN
-F 3 "" H 2500 4400 50  0001 C CNN
-	1    2500 4400
+P 2400 4400
+F 0 "#PWR01" H 2400 4150 50  0001 C CNN
+F 1 "GND" H 2400 4250 50  0000 C CNN
+F 2 "" H 2400 4400 50  0001 C CNN
+F 3 "" H 2400 4400 50  0001 C CNN
+	1    2400 4400
 	1    0    0    -1
 $EndComp
@@
 L power:PWR_FLAG #FLG04
 U 1 1 5A2856E5
-P 2300 4400
-F 0 "#FLG04" H 2300 4475 50  0001 C CNN
-F 1 "PWR_FLAG" H 2450 4550 50  0000 C CNN
-F 2 "" H 2300 4400 50  0001 C CNN
-F 3 "" H 2300 4400 50  0001 C CNN
-	1    2300 4400
+P 2200 4400
+F 0 "#FLG04" H 2200 4475 50  0001 C CNN
+F 1 "PWR_FLAG" H 2350 4550 50  0000 C CNN
+F 2 "" H 2200 4400 50  0001 C CNN
+F 3 "" H 2200 4400 50  0001 C CNN
+	1    2200 4400
 	-1   0    0    1
 $EndComp
@@
 D-
 $Comp
-L goldfish-rescue:USB_C_Receptacle-Connector J1
+L Connector:USB_C_Receptacle J1
 U 1 1 5A284C67
 P 2100 2600
@@
 	1800 4200 1800 4300
 Wire Wire Line
-	1800 4300 1900 4300
-Wire Wire Line
-	1900 4300 1900 4200
-Wire Wire Line
-	2000 4300 2000 4200
-Connection ~ 1900 4300
-Wire Wire Line
 	2100 4300 2100 4200
-Connection ~ 2000 4300
-Wire Wire Line
-	2200 4300 2200 4200
 Connection ~ 2100 4300
 Wire Wire Line
-	2300 4300 2300 4400
-Connection ~ 2200 4300
+	2200 4300 2200 4400
 Wire Wire Line
 	2800 1600 2700 1600
 Wire Wire Line
 	2800 1200 2800 1300
-Wire Wire Line
-	2700 1300 2800 1300
 Connection ~ 2800 1300
-Wire Wire Line
-	2800 1400 2700 1400
-Connection ~ 2800 1400
-Wire Wire Line
-	2800 1500 2700 1500
-Connection ~ 2800 1500
 Wire Wire Line
 	2700 1900 3000 1900
@@
 Connection ~ 2800 2400
 Wire Wire Line
-	2500 4300 2500 4400
-Connection ~ 2300 4300
+	2400 4300 2400 4400
+Connection ~ 2200 4300
 Wire Wire Line
 	3000 1300 3000 1200
@@
 	9050 1450 9300 1450
 Wire Wire Line
-	1900 4300 2000 4300
-Wire Wire Line
-	2000 4300 2100 4300
-Wire Wire Line
-	2100 4300 2200 4300
-Wire Wire Line
-	2200 4300 2300 4300
-Wire Wire Line
-	2800 1300 2800 1400
-Wire Wire Line
 	2800 1300 3000 1300
 Wire Wire Line
-	2800 1400 2800 1500
-Wire Wire Line
-	2800 1500 2800 1600
-Wire Wire Line
 	3400 1900 3400 2000
 Wire Wire Line
@@
 	2800 2400 2800 2500
 Wire Wire Line
-	2300 4300 2500 4300
+	2200 4300 2400 4300
 Wire Wire Line
 	7300 2700 7700 2700
@@
 PD5
 NoConn ~ 10350 3600
+Wire Wire Line
+	1800 4300 2100 4300
+Wire Wire Line
+	2100 4300 2200 4300
+Wire Wire Line
+	2800 1300 2800 1600
 $EndSCHEMATC
